File: hardware/commande_neons.sch (EAGLE design)
At the start: 16 parts

Commit message: Mise à jour des schéma
Parts:
- added C1, C2: 10u, resistor:C-EU025-024X044
- added CMD_LANC_PROG: (no value), switch-omron:31-XX
- added CN1, CN2, CN3, CN4, CN5, CN6, N1, N2, N3: 22-23-2021, con-molex:22-23-2021
- added LP, LP2: LED_PROG, con-molex:5566-6
- added R4, R5: 20k, resistor:R-EU_0204/5
- added R6, R7, R8: 500, resistor:R-EU_0204/7
- added X1: IN_CON1, con-garry:332-02
- added X2: IN_CON2, con-garry:332-02
- added X3: TO_CON1, con-garry:332-02
- added X4: TO_CON2, con-garry:332-02
- added X5, X6: 5566-4, con-molex:5566-4
Connections:
- new net N$17: ARDUINO_NANO1.D2, C1.1, R4.2
- new net N$18: R5.1, X2-2.S
- new net N$19: ARDUINO_NANO1.D3, C2.1, R5.2
- new net N$20: N3-2.S, NEON1.2
- new net N$21: R3.2, X5-1.S
- new net N$22: R2.2, X5-2.S
- new net N$23: R1.2, X5-3.S
- new net N$25: CN1-1.S, REL3.DS1
- new net N$26: CN1-2.S, CN4-2.S
- new net N$27: CN4-1.S, REL3.DS2
- new net N$28: CN2-1.S, REL2.DS1
- new net N$29: CN5-1.S, REL2.DS2
- new net N$30: CN2-2.S, CN5-2.S
- new net N$31: CN3-1.S, REL1.DS1
- new net N$32: CMD_PROG_NEON.P, X3-1.S
- new net N$33: CMD_PROG_NEON.S, X3-2.S
- new net N$34: CMD_LANC_PROG.P, X4-1.S
- new net N$35: CMD_LANC_PROG.S, X4-2.S
- new net N$36: LP-1.S, R8.2
- new net N$37: LP-3.S, R7.2
- new net N$38: LP-5.S, R6.2
- new net N$39: LED_P3.A, LP2-6.S
- new net N$40: LED_P3.C, LP2-5.S
- new net N$41: LED_P2.A, LP2-4.S
- new net N$42: LED_P2.C, LP2-3.S
- new net N$43: LED_P1.A, LP2-2.S
- new net N$44: LED_P1.C, LP2-1.S
- new net N$45: CN6-1.S, REL1.DS2
- new net N$46: CN3-2.S, CN6-2.S
- net AGND: now also N1-1.S, N2-1.S, N3-1.S; no longer REL1.DS2, REL2.DS2, REL3.DS2
- net GND: now also C1.2, C2.2, LP-2.S, LP-4.S, LP-6.S, X1-1.S, X2-1.S, X5-4.S; no longer CMD_PROG_NEON.S, LED_P1.C, LED_P2.C, LED_P3.C, REL1.K, REL2.K, REL3.K
- net N$1: now also ARDUINO_NANO1.D4; no longer ARDUINO_NANO1.D3
- net N$12: now also R4.1, X1-2.S; no longer ARDUINO_NANO1.D2, CMD_PROG_NEON.P
- net N$13: now also N2-2.S, NEON2.2; no longer NEON1.2, REL1.DS1
- net N$14: now also ARDUINO_NANO1.D7, R6.1; no longer ARDUINO_NANO1.D6, LED_P1.A
- net N$15: now also ARDUINO_NANO1.D8, R7.1; no longer ARDUINO_NANO1.D7, LED_P2.A
- net N$16: now also ARDUINO_NANO1.D9, R8.1; no longer ARDUINO_NANO1.D8, LED_P3.A
- net N$2: now also X6-2.S; no longer R1.2
- net N$3: now also REL1.K, REL2.K, REL3.K, X6-1.S; no longer R2.2, REL2.A
- net N$4: now also X6-4.S; no longer R3.2
- net N$5: now also ARDUINO_NANO1.D5; no longer ARDUINO_NANO1.D4
- net N$6: now also ARDUINO_NANO1.D6; no longer ARDUINO_NANO1.D5
- net N$7: now also N1-2.S; no longer REL3.DS1
- net N$9: now also REL2.A, X6-3.S; no longer NEON2.2, REL2.DS1
Other:
- note added: "CARTE PRINCIPALE"
- note removed: "CIRCUITS LOGIQUES"
- moved on the sheet: ARDUINO_NANO1, CMD_PROG_NEON, LED_P1, LED_P2, LED_P3, NEON1, NEON2, NEON3, R1, R2, R3, REL1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
